Commit message: More fixes. Cameras still not working inside gazebo.

File: src/etf_modules/sim_bringup/urdf/camera_depth_left.xacro (robot description, xacro)
@@ -12,5 +12,5 @@
                 <box size="0.04 0.1 0.04"/>
             </geometry>
-            <material name="grey"></material>
+            <!--<material name="grey"></material>-->
         </visual>
     </link>

File: src/etf_modules/sim_bringup/urdf/camera_depth_right.xacro (robot description, xacro)
@@ -12,5 +12,5 @@
                 <box size="0.04 0.1 0.04"/>
             </geometry>
-            <material name="grey"></material>
+            <!--<material name="grey"></material>-->
         </visual>
     </link>
